File: pcb/fc/kicad/fly-fc.kicad_pcb (KiCad board)
At the start: 2 copper layers, 46 x 44 mm, 35 parts, among them M1 8520 motor, M2 8520 motor, M3 8520 motor, M4 8520 motor, Q1 IRLB8721, Q2 IRLB8721, Q3 IRLB8721, Q4 IRLB8721, U2 GY-521 MPU6050

Commit message: Move the TPS63020 under the ESP32
The real module is about 27.5 x 18.7 mm, too big for the 20 x 12 mm spot
on the board. It now sits on foam under the ESP32 between its pin rows:
VIN and GND wires go to the rear IN and GND pads, OUT goes straight to
the ESP32 3V3 pin, which feeds the board through the front 3V3 pad.

- Board: removed the module outline, the OUT pad and its 3.3 V trace.
  Generator checks, netlist and KiCad DRC pass.
- Frame: checks that the module clears the MPU6050 (3.7 mm), C1, the
  ESP32 pin rows and the bridge tops; render updated.
- 3D model, build steps, pad tables, wiring and CLAUDE.md updated.

Co-Authored-By: Claude Opus 5.5 <noreply@anthropic.com>
Parts:
- removed J_OUT: wire pad, FlyDrone:J_OUT
Routing:
- net 3V3: track 44.4 -> 7.27 mm
Changed lines of the file:
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@@
     (pad "2" thru_hole circle (at 1.6 0) (size 2.5 2.5) (drill 1.2) (layers "*.Cu" "*.Mask") (remove_unused_layers no) (net 1 "GND"))
-  )
-  (footprint "FlyDrone:J_OUT"
-    (layer "F.Cu")
-    (at -2.54 18.5)
-    (property "Reference" "J_OUT" (at 0 -2.5 0) (layer "F.Fab") (effects (font (size 1 1) (thickness 0.15))))
-    (property "Value" "wire pad" (at 0 2.5 0) (layer "F.Fab") (effects (font (size 1 1) (thickness 0.15))))
-    (attr through_hole)
-    (pad "1" thru_hole circle (at 0 0) (size 1.6 1.6) (drill 0.8) (layers "*.Cu" "*.Mask") (remove_unused_layers no) (net 3 "3V3"))
   )
   (footprint "FlyDrone:J_TG"
@@
   (segment (start 5.08 -18.67) (end 5.08 -20.2) (width 0.3) (layer "F.Cu") (net 12))
   (segment (start 2.54 -20.2) (end 2.54 -14) (width 0.3) (layer "F.Cu") (net 1))
-  (segment (start -2.54 18.5) (end -2.54 16) (width 0.5) (layer "B.Cu") (net 3))
-  (segment (start -2.54 16) (end -8.89 9.65) (width 0.5) (layer "B.Cu") (net 3))
-  (segment (start -8.89 9.65) (end -8.89 -16) (width 0.5) (layer "B.Cu") (net 3))
   (zone (net 1) (net_name "GND") (layer "F.Cu") (name "GND F.Cu") (hatch edge 0.5)
     (priority 0)
@@
   (gr_line (start -11 -1.3) (end 11 -1.3) (stroke (width 0.18) (type solid)) (layer "F.SilkS"))
   (gr_line (start 11 -1.3) (end 11 -15.6) (stroke (width 0.18) (type solid)) (layer "F.SilkS"))
-  (gr_line (start -10 14.2) (end 10 14.2) (stroke (width 0.15) (type solid)) (layer "F.SilkS"))
-  (gr_line (start 10 14.2) (end 10 2.2) (stroke (width 0.15) (type solid)) (layer "F.SilkS"))
-  (gr_line (start 10 2.2) (end -10 2.2) (stroke (width 0.15) (type solid)) (layer "F.SilkS"))
-  (gr_line (start -10 2.2) (end -10 14.2) (stroke (width 0.15) (type solid)) (layer "F.SilkS"))
   (gr_poly (pts (xy 22.6 -2.44) (xy 22.6 -12.64) (xy 22 -12.64) (xy 22 -2.44)) (stroke (width 0.05) (type solid)) (fill solid) (layer "F.SilkS"))
   (gr_poly (pts (xy 16.7 -7.05) (xy 16.7 -7.85) (xy 14.1 -7.85) (xy 14.1 -7.05)) (stroke (width 0.05) (type solid)) (fill solid) (layer "F.SilkS"))
